Commit message: Corke IK

File: controllers/ur3_rtde_controller_IKPY/UR3e.urdf (robot description, URDF)
Before this commit: robot C:/mySciebo/_EMR25/github/emr25/urdf/UR3e.urdf, 18 links, 17 joints
Joints:
- removed joint hingejoint
- removed joint hingejoint_0
- removed joint hingejoint_1
- removed joint hingejoint_2
